Commit message: Added a new world, Aruco markers and Diff Drive

File: urdf/macro.xacro (robot description, xacro)
@@ -1,3 +1,3 @@
-<robot xmlns:xacro="http://www.ros.org/wiki/xacro">
+<robot xmlns:xacro="https://www.ros.org/wiki/xacro">
     <xacro:macro name="link_wheel" params="name">
         <link name="${name}">
@@ -10,5 +10,5 @@
               <origin rpy="0 1.5707 1.5707" xyz="0 0 0"/>
               <geometry>
-                <cylinder length="0.04" radius="0.1"/>
+                <cylinder length="0.01" radius="0.05"/>
               </geometry>
             </collision>
@@ -16,5 +16,5 @@
               <origin rpy="0 1.5707 1.5707" xyz="0 0 0"/>
               <geometry>
-                <cylinder length="0.04" radius="0.1"/>
+                <cylinder length="0.01" radius="0.05"/>
               </geometry>
             </visual>

File: urdf/mono_b.xacro (robot description, xacro)
@@ -7,13 +7,13 @@
   <!-- Chasis defined here -->
   <link name="link_chassis">
-    <pose>0 0 0.1 0 0 0</pose>
+    <pose>0 0 0 0 0 0</pose>
     <inertial>
-      <mass value="5"/>
-      <origin rpy="0 0 0" xyz="0 0 0.1"/>
-      <inertia ixx="0.0395416666667" ixy="0" ixz="0" iyy="0.106208333333" iyz="0" izz="0.106208333333"/>
+      <mass value="1"/>
+      <origin rpy="0 0 0" xyz="0 0 0"/>
+      <inertia ixx="0.0395416666667" ixy="0" ixz="0" iyy="0.206208333333" iyz="0" izz="0.106208333333"/>
     </inertial>
     <collision name="collision_chassis">
       <geometry>
-        <box size="0.5 0.3 0.07"/>
+			<cylinder length="0.03" radius="0.13"/>
       </geometry>
     </collision>
@@ -21,32 +21,65 @@
       <origin rpy="0 0 0" xyz="0 0 0"/>
       <geometry>
-        <box size="0.5 0.24 0.07"/>
+        	<cylinder length="0.03" radius="0.13"/>
       </geometry>
       <material name="blue"/>
     </visual>
+    </link>
     <!-- caster front -->
-    <collision name="caster_front_collision">
-      <origin rpy=" 0 0 0" xyz="0.35 0 -0.05"/>
+ 	<link name="chasis_to_caster_link">
+ 	<inertial>
+      <mass value="0.01"/>
+      <origin rpy="0 0 0" xyz="0 0 -0.0325"/>
+      <inertia ixx="0.1" ixy="0" ixz="0" iyy="0.1" iyz="0" izz="0.01"/>
+    </inertial>
+    <collision name="chasis_to_caster_collision">
+      <origin rpy=" 0 0 0" xyz="0 0 -0.0325"/>
       <geometry>
-        <sphere radius="0.05"/>
+        <cylinder length="0.055" radius="0.015"/>
       </geometry>
       <surface>
         <friction>
           <ode>
-            <mu>0</mu>
-            <mu2>0</mu2>
-            <slip1>1.0</slip1>
-            <slip2>1.0</slip2>
+            <mu>0.01</mu>
+            <mu2>0.01</mu2>
           </ode>
         </friction>
       </surface>
     </collision>
-    <visual name="caster_front_visual">
-      <origin rpy=" 0 0 0" xyz="0.2 0 -0.05"/>
+    <visual name="chasis_to_caster_visual">
+      <origin rpy=" 0 0 0" xyz="0 0 -0.0325"/>
       <geometry>
-        <sphere radius="0.05"/>
+        <cylinder length="0.055" radius="0.015"/>
       </geometry>
     </visual>
-    </link>
+ 	</link>
+ 	<!--// The SPHERE of the caster wheel is defined here -->
+    <link name="castor_wheel">
+ 		<inertial>
+          <mass value="0.5"/>
+          <origin rpy="0 0 0" xyz="0 0 0"/>
+          <inertia ixx="0.000526666666667" ixy="0" ixz="0" iyy="0.000526666666667" iyz="0" izz="0.000526666666667"/>
+        </inertial>
+        <collision name="link_caster_collision">
+        <origin rpy="0 0 0" xyz="0 0 0"/>
+          <geometry>
+            <sphere radius="0.015"/>
+          </geometry>
+          <surface>
+        <friction>
+          <ode>
+            <mu>0.1</mu>
+            <mu2>0.1</mu2>
+          </ode>
+        </friction>
+      </surface>
+        </collision>
+        <visual name="link_caster">
+          <origin rpy="0 0 0" xyz="0 0 0"/>
+          <geometry>
+            <sphere radius="0.015"/>
+          </geometry>
+        </visual>
+     </link>
    <!-- Camera -->
   <link name="camera_link">
@@ -54,5 +87,5 @@
       <origin xyz="0 0 0" rpy="0 0 0"/>
       <geometry>
-    <box size="0.02 0.16 0.15"/>
+      <box size="0.01 0.06 0.06"/>
       </geometry>
     </collision>
@@ -60,7 +93,8 @@
       <origin xyz="0 0 0" rpy="0 0 0"/>
       <geometry>
-    <box size="0.02 0.16 0.15"/>
+        <!-- <mesh filename="package://mono_bot/meshes/camera_box.dae" scale="1 1 1"/> -->
+        <mesh filename="package://mono_bot/meshes/$(arg aruco_id)" scale="3 3 3"/>
+        <!-- <box size="0.01 0.16 0.15"/>       -->
       </geometry>
-      <material name="red"/>
     </visual>
     <inertial>
@@ -70,15 +104,54 @@
     </inertial>
   </link>
- <joint name="camera_joint" type="fixed">
+  <joint name="camera_joint" type="fixed">
     <axis xyz="0 1 0" />
-    <origin xyz="0.15 0 0.035" rpy="0 0 0"/>
+    <origin xyz="0.05 0 0.115" rpy="0 0 0"/>
     <parent link="link_chassis"/>
     <child link="camera_link"/>
   </joint>
+  <link name="camera_link_2">
+    <collision>
+      <origin xyz="0 0 0" rpy="0 0 0"/>
+      <geometry>
+        <box size="0.01 0.06 0.06"/>
+      </geometry>
+    </collision>
+    <visual>
+      <origin xyz="0 0 0" rpy="0 0 0"/>
+      <geometry>
+        <mesh filename="package://mono_bot/meshes/$(arg aruco_id)" scale="3 3 3"/>
+    	  <!-- <box size="0.01 0.08 0.16"/> -->
+      </geometry>
+    </visual>
+    <inertial>
+      <mass value="1e-5" />
+      <origin xyz="0 0 0" rpy="0 0 0"/>
+      <inertia ixx="1e-6" ixy="0" ixz="0" iyy="1e-6" iyz="0" izz="1e-6" />
+    </inertial>
+  </link>
+  <joint name="camera_joint_2" type="fixed">
+    <axis xyz="0 1 0" />
+    <origin xyz="-0.05 0 0.115" rpy="0 0 3.14"/>
+    <parent link="link_chassis"/>
+    <child link="camera_link_2"/>
+  </joint>
+  <joint name="chasis_to_cylinder_joint" type="continuous">
+   	<axis rpy="0 0 0" xyz="0 0 1" />
+    <origin xyz="0.085 0 -0.015" rpy="0 0 0"/>
+    <parent link="link_chassis"/>
+    <child link="chasis_to_caster_link"/>
+  </joint>
+  <joint name="cylinder_to_caster_joint" type="continuous">
+  	<axis rpy="0 0 0" xyz="0 1 0" />
+    <origin xyz="0.01 0 -0.065" rpy="0 0 0"/>
+    <!-- origin xyz="0 0 0" rpy="0 0 0"/-->
+    <parent link="chasis_to_caster_link"/>
+    <child link="castor_wheel"/>
+  </joint>
   <!-- Create wheel right -->
    <xacro:link_wheel name="link_right_wheel" />
-   <xacro:joint_wheel name="joint_right_wheel"  child="link_right_wheel"  origin_xyz="-0.08 0.12 0"  />
+   <xacro:joint_wheel name="joint_right_wheel"  child="link_right_wheel"  origin_xyz="-0.07 0.145 -0.045"  />
   <!-- Left Wheel link -->
   <xacro:link_wheel name="link_left_wheel" />
-  <xacro:joint_wheel name="joint_left_wheel"   child="link_left_wheel"   origin_xyz="-0.08 -0.12 0"  />
+  <xacro:joint_wheel name="joint_left_wheel"   child="link_left_wheel"   origin_xyz="-0.07 -0.145 -0.045"  />
 </robot>
