Commit message: Correted the aruco box. Detection works now after using correct dictionary 4X4

File: urdf/mono_b.xacro (robot description, xacro)
@@ -91,8 +91,9 @@
     </collision>
     <visual>
-      <origin xyz="0 0 0" rpy="0 0 0"/>
+      <!-- FRONT Facing camera -->
+      <origin xyz="0 0 0" rpy="3.14 0 0"/>
       <geometry>
         <!-- <mesh filename="package://mono_bot/meshes/camera_box.dae" scale="1 1 1"/> -->
-        <mesh filename="package://mono_bot/meshes/$(arg aruco_id)" scale="3 3 3"/>
+        <mesh filename="package://mono_bot/meshes/$(arg aruco_id)" scale="2 2 2"/>
         <!-- <box size="0.01 0.16 0.15"/>       -->
       </geometry>
@@ -106,5 +107,5 @@
   <joint name="camera_joint" type="fixed">
     <axis xyz="0 1 0" />
-    <origin xyz="0.05 0 0.115" rpy="0 0 0"/>
+    <origin xyz="0.05 0 0.140" rpy="0 0 0"/>
     <parent link="link_chassis"/>
     <child link="camera_link"/>
@@ -118,7 +119,8 @@
     </collision>
     <visual>
-      <origin xyz="0 0 0" rpy="0 0 0"/>
+      <!-- BACK Facing camera -->
+      <origin xyz="0 0 0" rpy="3.14 0 0"/>
       <geometry>
-        <mesh filename="package://mono_bot/meshes/$(arg aruco_id)" scale="3 3 3"/>
+        <mesh filename="package://mono_bot/meshes/$(arg aruco_id)" scale="2 2 2"/>
     	  <!-- <box size="0.01 0.08 0.16"/> -->
       </geometry>
@@ -132,5 +134,5 @@
   <joint name="camera_joint_2" type="fixed">
     <axis xyz="0 1 0" />
-    <origin xyz="-0.05 0 0.115" rpy="0 0 3.14"/>
+    <origin xyz="-0.05 0 0.140" rpy="0 0 3.14"/>
     <parent link="link_chassis"/>
     <child link="camera_link_2"/>
